Commit message: Created Cards

File: src/drivers/universal_robot/ur_description/urdf/block.urdf (robot description, URDF)
Before this commit: robot block, 1 links, 0 joints
Links:
- link base_link: geometry collision box size=0.10 0.045 0.0025; visual box size=0.10 0.045 0.0025

Commit message: Fixed Card urdf

File: src/drivers/universal_robot/ur_description/urdf/block.urdf (robot description, URDF)
Before this commit: robot block, 1 links, 0 joints
Links:
- link base_link: mass 0.0225 -> 0.4
